File: schematic/ESP32_module.sch (KiCad schematic (older format))
At the start: 26 parts, among them J1 Conn_02x03_Odd_Even, J14 Conn_01x11_Male, J2 Conn_02x05_Odd_Even, J3 Conn_02x06_Odd_Even, U1 ESP32-WROOM-32

Commit message: wireing
Parts:
- J1: footprint Connector_PinHeader_1.27mm:PinHeader_2x03_P1.27mm_Vertical_SMD -> Apsu:PinHeader_2x03_P1.27mm_Vertical_IDC
Changed lines of the file:
@@
 F 0 "J1" H 5900 2067 50  0000 C CNN
 F 1 "Conn_02x03_Odd_Even" H 5900 1976 50  0000 C CNN
-F 2 "Connector_PinHeader_1.27mm:PinHeader_2x03_P1.27mm_Vertical_SMD" H 5850 1750 50  0001 C CNN
+F 2 "Apsu:PinHeader_2x03_P1.27mm_Vertical_IDC" H 5850 1750 50  0001 C CNN
 F 3 "~" H 5850 1750 50  0001 C CNN
 	1    5850 1750

Commit message: added MPN
Parts:
- C1, C22, C3: MPN (none) -> C0805C104J5RACTU
- C2: MPN (none) -> C0805C226K9PACTU
- C23: MPN (none) -> C0805C106K8PACTU
- R1, R16, R2, R24, R25, R3, R4, R5, R6, R7: MPN (none) -> ERA-6AEB103V
- R12: MPN (none) -> ERA-6AEB104V
- R13: MPN (none) -> ERA6AEB4991V
- R27, R28, R29, R30: MPN (none) -> ERA6AEB101V
- U1: MPN (none) -> ESP32-WROOM-32D

Commit message: added MPN for connectors
Parts:
- J1: MPN (none) -> GRPB032VWVN-RC
- J2: MPN (none) -> 3220-10-0100-00
- J3: MPN (none) -> BHR-12-VUA
