File: schematic/communication.sch (KiCad schematic (older format))
At the start: 12 parts, among them J12 Conn_01x02_Male, J13 Conn_01x02, U8 SP3485CN

Commit message: added MPN for connectors
Parts:
- J13: MPN (none) -> B2B-XH-A(LF)(SN)
